File: IVO build V6.2/IVO build V6.2.kicad_pcb (KiCad board)
At the start: 0 parts

Commit message: Updated schematic
Parts:
- added Q2: C2M0080120D, Package_TO_SOT_THT:TO-247-3_Vertical, F.Cu at (136.2, 87.0)
- added U2: 1EDI60I12AF, Package_SO:SOIC-8_3.9x4.9mm_P1.27mm, F.Cu at (98.3, 103.2)
- added U3: MGJ1D121505MPC-R7, footprints:MGJ1_MUR, F.Cu at (122.5, 94.4)
Routing:
- net Net-(U2-VCC2): track 0.00 -> 30.1 mm
- net Net-(Q2-S): track 0.00 -> 22.6 mm
Other:
- board outline added: 75.5 x 40.6 mm
- copper layers 0 -> 2
