File: IVO build V6.2/IVO build V6.2.kicad_pcb (KiCad board)
At the start: 2 copper layers, 75.5 x 40.6 mm, 3 parts, among them Q2 C2M0080120D, U2 1EDI60I12AF, U3 MGJ1D121505MPC-R7

Commit message: Updated schematic
Connections:
- U3 pad 4: unconnected-(U3--VOUT-Pad4) -> Net-(C11-Pad2)
Changed lines of the file:
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@@
   (net 13 "unconnected-(U3-NC-Pad2)")
   (net 14 "unconnected-(U3--VIN-Pad1)")
-  (net 15 "unconnected-(U3--VOUT-Pad4)")
-  (net 16 "Net-(U1-IN)")
+  (net 15 "Net-(C11-Pad2)")
+  (net 16 "Net-(U3-+VIN)")
   (net 17 "unconnected-(U3-NC-Pad7)")
   (footprint "Package_TO_SOT_THT:TO-247-3_Vertical" (layer "F.Cu")
@@
     )
     (pad "4" smd rect (at -6.985 7.1125) (size 2.3114 0.9906) (layers "F.Cu" "F.Paste" "F.Mask")
-      (net 15 "unconnected-(U3--VOUT-Pad4)") (pinfunction "-VOUT") (pintype "power_in")
+      (net 15 "Net-(C11-Pad2)") (pinfunction "-VOUT") (pintype "power_in")
     )
     (pad "5" smd rect (at 6.985 7.1125) (size 2.3114 0.9906) (layers "F.Cu" "F.Paste" "F.Mask")
@@
     )
     (pad "8" smd rect (at 6.985 -8.8895) (size 2.3114 0.9906) (layers "F.Cu" "F.Paste" "F.Mask")
-      (net 16 "Net-(U1-IN)") (pinfunction "+VIN") (pintype "power_in")
+      (net 16 "Net-(U3-+VIN)") (pinfunction "+VIN") (pintype "power_in")
     )
   )
