File: IVO build V6.2/IVO build V6.2.kicad_pcb (KiCad board)
At the start: 2 copper layers, 75.5 x 40.6 mm, 3 parts, among them Q2 C2M0080120D, U2 1EDI60I12AF, U3 MGJ1D121505MPC-R7

Commit message: Updated schematic
Parts:
- added U1: L7805, Package_TO_SOT_THT:TO-92, F.Cu at (95.0, 85.3)
Changed lines of the file:
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@@
 	(net 13 "unconnected-(U3-NC-Pad2)")
 	(net 14 "unconnected-(U3--VIN-Pad1)")
-	(net 15 "Net-(C11-Pad2)")
+	(net 15 "Net-(C12-Pad2)")
 	(net 16 "Net-(U3-+VIN)")
 	(net 17 "unconnected-(U3-NC-Pad7)")
+	(net 18 "+12V")
 	(footprint "Package_TO_SOT_THT:TO-247-3_Vertical"
 		(layer "F.Cu")
@@
 		)
 		(property ki_fp_filters "TO?247*")
+		(sheetname "Root")
 		(sheetfile "IVO build V6.2.kicad_sch")
 		(attr through_hole)
@@
 		)
 		(property "Value" "MGJ1D121505MPC-R7"
-			(at 0 0 0)
-			(unlocked yes)
-			(layer "F.Fab")
+			(at 0.3302 2.0833 0)
+			(unlocked yes)
+			(layer "F.Fab")
+			(hide yes)
 			(effects
 				(font
@@
 		)
 		(property ki_fp_filters "MGJ1_MUR")
+		(sheetname "Root")
 		(sheetfile "IVO build V6.2.kicad_sch")
 		(attr smd)
@@
 			(size 2.3114 0.9906)
 			(layers "F.Cu" "F.Paste" "F.Mask")
-			(net 15 "Net-(C11-Pad2)")
+			(net 15 "Net-(C12-Pad2)")
 			(pinfunction "-VOUT")
 			(pintype "power_in")
@@
 			(pinfunction "+VIN")
 			(pintype "power_in")
+		)
+	)
+	(footprint "Package_TO_SOT_THT:TO-92"
+		(layer "F.Cu")
+		(at 94.996 85.2932)
+		(descr "TO-92 leads molded, narrow, drill 0.75mm (see NXP sot054_po.pdf)")
+		(tags "to-92 sc-43 sc-43a sot54 PA33 transistor")
+		(property "Reference" "U1"
+			(at 1.27 -3.56 0)
+			(layer "F.SilkS")
+			(effects
+				(font
+					(size 1 1)
+					(thickness 0.15)
+				)
+			)
+		)
+		(property "Value" "L7805"
+			(at 1.27 2.79 0)
+			(layer "F.Fab")
+			(effects
+				(font
+					(size 1 1)
+					(thickness 0.15)
+				)
+			)
+		)
+		(property "Footprint" "Package_TO_SOT_THT:TO-92"
+			(at 0 0 0)
+			(unlocked yes)
+			(layer "F.Fab")
+			(hide yes)
+			(effects
+				(font
+					(size 1.27 1.27)
+				)
+			)
+		)
+		(property "Datasheet" "http://www.st.com/content/ccc/resource/technical/document/datasheet/41/4f/b3/b0/12/d4/47/88/CD00000444.pdf/files/CD00000444.pdf/jcr:content/translations/en.CD00000444.pdf"
+			(at 0 0 0)
+			(unlocked yes)
+			(layer "F.Fab")
+			(hide yes)
+			(effects
+				(font
+					(size 1.27 1.27)
+				)
+			)
+		)
+		(property "Description" "Positive 1.5A 35V Linear Regulator, Fixed Output 5V, TO-220/TO-263/TO-252"
+			(at 0 0 0)
+			(unlocked yes)
+			(layer "F.Fab")
+			(hide yes)
+			(effects
+				(font
+					(size 1.27 1.27)
+				)
+			)
+		)
+		(property ki_fp_filters "TO?252* TO?263* TO?220*")
+		(sheetname "Root")
+		(sheetfile "IVO build V6.2.kicad_sch")
+		(attr through_hole)
+		(fp_line
+			(start -0.53 1.85)
+			(end 3.07 1.85)
+			(stroke
+				(width 0.12)
+				(type solid)
+			)
+			(layer "F.SilkS")
+		)
+		(fp_arc
+			(start -0.568478 1.838478)
+			(mid -1.132087 -0.994977)
+			(end 1.27 -2.6)
+			(stroke
+				(width 0.12)
+				(type solid)
+			)
+			(layer "F.SilkS")
+		)
+		(fp_arc
+			(start 1.27 -2.6)
+			(mid 3.672087 -0.994977)
+			(end 3.108478 1.838478)
+			(stroke
+				(width 0.12)
+				(type solid)
+			)
+			(layer "F.SilkS")
+		)
+		(fp_line
+			(start -1.46 -2.73)
+			(end -1.46 2.01)
+			(stroke
+				(width 0.05)
+				(type solid)
+			)
+			(layer "F.CrtYd")
+		)
+		(fp_line
+			(start -1.46 -2.73)
+			(end 4 -2.73)
+			(stroke
+				(width 0.05)
+				(type solid)
+			)
+			(layer "F.CrtYd")
+		)
+		(fp_line
+			(start 4 2.01)
+			(end -1.46 2.01)
+			(stroke
+				(width 0.05)
+				(type solid)
+			)
+			(layer "F.CrtYd")
+		)
+		(fp_line
+			(start 4 2.01)
+			(end 4 -2.73)
+			(stroke
+				(width 0.05)
+				(type solid)
+			)
+			(layer "F.CrtYd")
+		)
+		(fp_line
+			(start -0.5 1.75)
+			(end 3 1.75)
+			(stroke
+				(width 0.1)
+				(type solid)
+			)
+			(layer "F.Fab")
+		)
+		(fp_arc
+			(start -0.483625 1.753625)
+			(mid -1.021221 -0.949055)
+			(end 1.27 -2.48)
+			(stroke
+				(width 0.1)
+				(type solid)
+			)
+			(layer "F.Fab")
+		)
+		(fp_arc
+			(start 1.27 -2.48)
+			(mid 3.561221 -0.949055)
+			(end 3.023625 1.753625)
+			(stroke
+				(width 0.1)
+				(type solid)
+			)
+			(layer "F.Fab")
+		)
+		(fp_text user "${REFERENCE}"
+			(at 1.27 0 0)
+			(layer "F.Fab")
+			(effects
+				(font
+					(size 1 1)
+					(thickness 0.15)
+				)
+			)
+		)
+		(pad "1" thru_hole rect
+			(at 0 0)
+			(size 1.3 1.3)
+			(drill 0.75)
+			(layers "*.Cu" "*.Mask")
+			(remove_unused_layers no)
+			(net 18 "+12V")
+			(pinfunction "IN")
+			(pintype "power_in")
+		)
+		(pad "2" thru_hole circle
+			(at 1.27 -1.27)
+			(size 1.3 1.3)
+			(drill 0.75)
+			(layers "*.Cu" "*.Mask")
+			(remove_unused_layers no)
+			(net 9 "GND")
+			(pinfunction "GND")
+			(pintype "power_in")
+		)
+		(pad "3" thru_hole circle
+			(at 2.54 0)
+			(size 1.3 1.3)
+			(drill 0.75)
+			(layers "*.Cu" "*.Mask")
+			(remove_unused_layers no)
+			(net 10 "Net-(U1-OUT)")
+			(pinfunction "OUT")
+			(pintype "power_out")
+		)
+		(model "${KICAD6_3DMODEL_DIR}/Package_TO_SOT_THT.3dshapes/TO-92.wrl"
+			(offset
+				(xyz 0 0 0)
+			)
+			(scale
+				(xyz 1 1 1)
+			)
+			(rotate
+				(xyz 0 0 0)
+			)
 		)
 	)
@@
 		)
 		(property ki_fp_filters "SOIC*3.9x4.9mm*P1.27mm*")
+		(sheetname "Root")
 		(sheetfile "IVO build V6.2.kicad_sch")
 		(attr smd)

Commit message: updated schematic and added picture
Parts:
- U3: moved to B.Cu
- turned U3 to 180 degrees
Routing:
- net GND: track 0.00 -> 22.6 mm
- net Net-(U1-OUT): track 0.00 -> 18.5 mm
- net Net-(Q2-S): track 22.6 -> 36.6 mm
- net Net-(U2-VCC2): track 30.1 -> 35.3 mm, vias 0 -> 1
