File: IVO build V6.2/IVO build V6.2.kicad_sch (KiCad schematic)
At the start: 15 parts, among them Q2 C2M0080120D, U1 L7805, U2 1EDI60I12AF, U3 MGJ1D121505MPC-R7

Commit message: Updated schematic
Parts:
- R1, R2: value 10 ohm 5 Watt -> 10 ohm 1 Watt
- U1: footprint (none) -> Package_TO_SOT_THT:TO-92
Changed lines of the file:
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@@
 			)
 		)
-		(property "Footprint" ""
+		(property "Footprint" "Package_TO_SOT_THT:TO-92"
 			(at 126.365 81.28 0)
 			(effects
@@
 			)
 		)
-		(property "Value" "10 ohm  5 Watt"
+		(property "Value" "10 ohm  1 Watt"
 			(at 200.66 68.58 90)
 			(effects
@@
 			)
 		)
-		(property "Value" "10 ohm  5 Watt"
+		(property "Value" "10 ohm  1 Watt"
 			(at 200.66 53.34 90)
 			(effects

Commit message: updated schematic and added picture
Parts:
- added C2, C3, C4: 100nF, symbol Device:C
- added D1: 2CL77, symbol Device:D
- added L2, L3, L4: ~, symbol Device:L
- added TP1: TestPoint, symbol Connector:TestPoint
- added TP2: bridge, symbol Connector:TestPoint
Connections:
- net +12V: now also Q2.2 (D)
- net at C1.2, C10.2, C12.1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: now also L2.1, TP2.1; no longer Q2.3 (S)
- new net: C2.1, C3.1, D1.2 (A), L3.2, Q2.3 (S), TP1.1
- new net: C3.2, L3.1
- new net: C2.2, C4.1, D1.1 (K), L2.2, L4.1
- new net: C4.2, L4.2
Other:
- note added: "Outside board"
- moved on the sheet: Q2
